Commit message: 1.resume to use urdf.xacro 2.change the shape.position,size of link 3.add rviz config file

File: simple_robot_description/urdf/simple_robot.urdf (robot description, URDF)
Before this commit: robot simple_robot, 2 links, 1 joints
Links:
- link base_link: geometry visual box size=0.2 0.2 0.1
- link moving_link: geometry visual box size=0.1 0.5 0.1

File: simple_robot_description/urdf/simple_robot.urdf.xacro (robot description, xacro)
@@ -1,11 +1,27 @@
 <?xml version="1.0"?>
 <robot xmlns:xacro="http://www.ros.org/wiki/xacro" name="simple_robot">
-    <link name="base_link"/>
+    <material name="bright_red">
+        <color rgba="1.0 0.0 0.0 1.0"/>
+    </material>
+    <material name="bright_blue">
+        <color rgba="0.0 0.0 1.0 1.0"/>
+    </material>
+    <link name="base_link">
+        <visual>
+            <origin xyz="0 0 0.025" rpy="0 0 0"/>
+            <geometry>
+                <!-- cylinder radius="0.2" length="0.05"/ -->
+                <box size="0.2 0.2 0.1"/>
+            </geometry>
+            <material name="bright_blue"/>
+        </visual>
+    </link>
     <link name="moving_link">
         <visual>
+            <origin xyz="0 0.3 0" rpy="0 0 0"/>
             <geometry>
-                <box size="0.1 0.1 0.5"/>
+                <box size="0.1 0.5 0.1"/>
             </geometry>
-            <origin xyz="0 0 0.25"/>
+            <material name="bright_red"/>
         </visual>
     </link>
@@ -13,6 +29,7 @@
         <parent link="base_link"/>
         <child link="moving_link"/>
-        <origin xyz="0 0 0" rpy="0 0 0"/>
-        <axis xyz="0 0 1"/> <limit lower="-3.14" upper="3.14" effort="10.0" velocity="1.0"/>
+        <origin xyz="0 0 0.05" rpy="0 0 0"/>
+        <axis xyz="0 0 1"/>
+        <limit lower="-3.14" upper="3.14" effort="10.0" velocity="1.0"/>
     </joint>
     <ros2_control name="MockHardware" type="system">
