Commit message: fine tune joints and links' axis and size

File: simple_robot_description2/urdf/simple_robot.urdf.xacro (robot description, xacro)
@@ -12,8 +12,8 @@
     <link name="base_link">
         <visual>
-            <origin xyz="0 0 0.025" rpy="0 0 0"/>
+            <origin xyz="0 0 0" rpy="0 0 0"/>
             <geometry>
                 <!-- cylinder radius="0.2" length="0.05"/ -->
-                <box size="0.2 0.2 0.1"/>
+                <box size="0.2 0.2 0.2"/>
             </geometry>
             <material name="bright_blue"/>
@@ -24,5 +24,5 @@
             <origin xyz="0 0.3 0" rpy="0 0 0"/>
             <geometry>
-                <box size="0.1 0.5 0.1"/>
+                <box size="0.2 0.6 0.2"/>
             </geometry>
             <material name="bright_red"/>
@@ -31,7 +31,7 @@
     <link name="moving_link2">
         <visual>
-            <origin xyz="0 0.8 0" rpy="0 0 0"/>
+            <origin xyz="0 0.3 0" rpy="0 0 0"/>
             <geometry>
-                <box size="0.1 0.5 0.1"/>
+                <box size="0.2 0.6 0.2"/>
             </geometry>
             <material name="bright_green"/>
@@ -41,5 +41,5 @@
         <parent link="base_link"/>
         <child link="moving_link"/>
-        <origin xyz="0 0 0.05" rpy="0 0 0"/>
+        <origin xyz="0 0.1 0" rpy="0 0 0"/>
         <axis xyz="0 0 1"/>
         <limit lower="-3.14" upper="3.14" effort="10.0" velocity="1.0"/>
@@ -48,5 +48,5 @@
         <parent link="moving_link"/>
         <child link="moving_link2"/>
-        <origin xyz="0 0 0.05" rpy="0 0 0"/>
+        <origin xyz="0 0.6 0" rpy="0 0 0"/>
         <axis xyz="0 0 1"/>
         <limit lower="-3.14" upper="3.14" effort="10.0" velocity="1.0"/>
